Commit message: add boat related models

File: vrx_urdf/wamv_description/urdf/wamv_base.urdf.xacro (robot description, xacro)
@@ -8,5 +8,5 @@
     <!-- Main float -->
     <collision name="${prefix}_float">
-      <origin xyz="-0.4 ${1.03*reflect} 0.2" rpy="${0*reflect} 1.57 0" />
+      <origin xyz="-0.4 ${1.03*reflect} 0.3" rpy="${0*reflect} 1.57 0" />
       <geometry>
         <cylinder length="4" radius="0.2" />

File: vrx_urdf/wamv_gazebo/urdf/wamv_gazebo.urdf.xacro (robot description, xacro)
@@ -121,12 +121,4 @@
       <xacro:wamv_p3d name="p3d_wamv"/>
     </xacro:if>
-    <!-- Add pinger -->
-    <xacro:if value="$(arg pinger_enabled)">
-      <xacro:wamv_pinger sensor_name="receiver" position="-528 191 -2.0" />
-    </xacro:if>
-    <!-- Add ball shooter (default pitch angle: ~-60 deg) -->
-    <xacro:if value="$(arg ball_shooter_enabled)">
-      <xacro:wamv_ball_shooter name="ball_shooter" x="0.54" y="0.30" z="1.296" pitch="-1.04"/>
-    </xacro:if>
     <!-- ==== VRX sensor configuration ==== -->
     <xacro:if value="$(arg vrx_sensors_enabled)">
@@ -145,8 +137,4 @@
       <!-- Add 3D LIDAR -->
       <xacro:lidar name="lidar_wamv" type="16_beam"/>
-      <!-- Add pinger -->
-      <xacro:wamv_pinger sensor_name="receiver" position="-528 191 -2.0" />
-      <!-- Add ball shooter (default pitch angle: ~-60 deg) -->
-      <xacro:wamv_ball_shooter name="ball_shooter" x="0.54" y="0.30" z="1.296" pitch="-1.04"/>
     </xacro:if>
   </xacro:unless>
